File: RTK1010Board.kicad_sch (KiCad schematic)
At the start: 75 parts, among them J1 SMA, J2 IPEX, J3 USB_OTG, J4 BNO055, U1 RTK-1010, U2 NCP1117-3.3_SOT223, U3 MCP1700-3302E_SOT23, U4 ESP32-S2-WROVER

Commit message: ibom added
Parts:
- C12, C2, C8, C9, J3, R13, R14, R15, R16, R4, R5: Variant (none) -> B
- C13, C5, J2, L1, U1: Variant (none) -> A,B
- L3: value ?H -> 1.2uH; Variant (none) -> A,B
- R7, R8, XA1: Variant (none) -> A
Changed lines of the file:
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@@
+      (effects (font (size 1.27 1.27)) hide)
+    )
+    (property "Variant" "A,B" (id 4) (at 19.05 60.96 0)
       (effects (font (size 1.27 1.27)) hide)
     )
@@
     )
     (property "Value" "100nF" (id 1) (at 64.77 106.6799 0)
-      (effects (font (size 1.27 1.27)) (justify left) hide)
+      (effects (font (size 1.27 1.27)) (justify left))
     )
     (property "Footprint" "Capacitor_SMD:C_0805_2012Metric_Pad1.18x1.45mm_HandSolder" (id 2) (at 61.9252 109.22 0)
@@
     )
     (property "Datasheet" "~" (id 3) (at 60.96 105.41 0)
+      (effects (font (size 1.27 1.27)) hide)
+    )
+    (property "Variant" "B" (id 4) (at 60.96 105.41 0)
       (effects (font (size 1.27 1.27)) hide)
     )
@@
     )
     (property "Datasheet" "" (id 3) (at 64.77 39.37 0)
+      (effects (font (size 1.27 1.27)) hide)
+    )
+    (property "Variant" "A,B" (id 4) (at 64.77 39.37 0)
       (effects (font (size 1.27 1.27)) hide)
     )
@@
       (effects (font (size 1.27 1.27)) hide)
     )
+    (property "Variant" "A" (id 4) (at 163.83 25.4 90)
+      (effects (font (size 1.27 1.27)) hide)
+    )
     (pin "1")
     (pin "2")
@@
       (effects (font (size 1.27 1.27)) hide)
     )
+    (property "Variant" "B" (id 4) (at 57.15 116.84 0)
+      (effects (font (size 1.27 1.27)) hide)
+    )
     (pin "1")
     (pin "2")
@@
       (effects (font (size 1.27 1.27)) hide)
     )
+    (property "Variant" "" (id 4) (at 107.95 77.47 90)
+      (effects (font (size 1.27 1.27)) hide)
+    )
     (pin "1")
     (pin "2")
@@
       (effects (font (size 1.27 1.27)) hide)
     )
+    (property "Variant" "B" (id 4) (at 57.15 181.61 0)
+      (effects (font (size 1.27 1.27)) hide)
+    )
     (pin "1")
     (pin "2")
@@
     (property "Datasheet" "" (id 3) (at 260.35 -45.72 0)
       (effects (font (size 1.524 1.524)) hide)
+    )
+    (property "Variant" "A" (id 4) (at 214.63 49.53 0)
+      (effects (font (size 1.27 1.27)) hide)
     )
     (pin "3V3")
@@
       (effects (font (size 1.27 1.27)) hide)
     )
+    (property "Variant" "B" (id 4) (at 168.91 137.16 0)
+      (effects (font (size 1.27 1.27)) hide)
+    )
     (pin "1")
     (pin "2")
@@
       (effects (font (size 1.27 1.27)) (justify left))
     )
-    (property "Value" "?H" (id 1) (at 49.53 39.37 0)
+    (property "Value" "1.2uH" (id 1) (at 49.53 39.37 0)
       (effects (font (size 1.27 1.27)) (justify left))
     )
@@
       (effects (font (size 1.27 1.27)) hide)
     )
-    (property "Datasheet" "~" (id 3) (at 45.72 43.18 0)
+    (property "Datasheet" "https://www.reichelt.de/smd-induktivitaet-0805-keramik-1-2-h-l-0805as-1-2--p255497.html?&trstct=pol_0&nbc=1" (id 3) (at 45.72 43.18 0)
+      (effects (font (size 1.27 1.27)) hide)
+    )
+    (property "Variant" "A,B" (id 4) (at 45.72 43.18 0)
       (effects (font (size 1.27 1.27)) hide)
     )
@@
       (effects (font (size 1.27 1.27)) hide)
     )
+    (property "Variant" "A" (id 4) (at 170.18 22.86 90)
+      (effects (font (size 1.27 1.27)) hide)
+    )
     (pin "1")
     (pin "2")
@@
       (effects (font (size 1.27 1.27)) hide)
     )
+    (property "Variant" "A,B" (id 4) (at 111.76 53.34 0)
+      (effects (font (size 1.27 1.27)) hide)
+    )
     (pin "1")
     (pin "2")
   )
   (symbol (lib_id "Device:C") (at 148.59 144.78 0) (unit 1)
-    (in_bom yes) (on_board yes) (fields_autoplaced)
-    (property "Reference" "C2" (id 0) (at 152.4 143.5099 0)
-      (effects (font (size 1.27 1.27)) (justify left))
-    )
-    (property "Value" "100nF" (id 1) (at 152.4 146.0499 0)
-      (effects (font (size 1.27 1.27)) (justify left) hide)
+    (in_bom yes) (on_board yes)
+    (property "Reference" "C2" (id 0) (at 149.86 142.24 0)
+      (effects (font (size 1.27 1.27)) (justify left))
+    )
+    (property "Value" "100nF" (id 1) (at 148.59 139.7 0)
+      (effects (font (size 1.27 1.27)) (justify left))
     )
     (property "Footprint" "Capacitor_SMD:C_0805_2012Metric_Pad1.18x1.45mm_HandSolder" (id 2) (at 149.5552 148.59 0)
@@
     )
     (property "Datasheet" "~" (id 3) (at 148.59 144.78 0)
+      (effects (font (size 1.27 1.27)) hide)
+    )
+    (property "Variant" "B" (id 4) (at 148.59 144.78 0)
       (effects (font (size 1.27 1.27)) hide)
     )
@@
       (effects (font (size 1.27 1.27)) hide)
     )
+    (property "Variant" "B" (id 4) (at 138.43 149.86 90)
+      (effects (font (size 1.27 1.27)) hide)
+    )
     (pin "1")
     (pin "2")
@@
     )
     (property "Datasheet" "https://www.reichelt.de/usb-buchse-typ-micro-b-smd-gull-wing-mpe-712-1-s-bs0-p263308.html?&trstct=pol_1&nbc=1" (id 3) (at 158.75 151.13 0)
+      (effects (font (size 1.27 1.27)) hide)
+    )
+    (property "Variant" "B" (id 4) (at 162.56 149.86 0)
       (effects (font (size 1.27 1.27)) hide)
     )
@@
     )
     (property "Datasheet" "~" (id 3) (at 138.43 152.4 0)
+      (effects (font (size 1.27 1.27)) hide)
+    )
+    (property "Variant" "B" (id 4) (at 138.43 152.4 90)
       (effects (font (size 1.27 1.27)) hide)
     )
@@
       (effects (font (size 1.27 1.27)) hide)
     )
+    (property "Variant" "A,B" (id 4) (at 30.48 60.96 0)
+      (effects (font (size 1.27 1.27)) hide)
+    )
     (pin "1")
     (pin "2")
@@
       (effects (font (size 1.27 1.27)) hide)
     )
+    (property "Variant" "B" (id 4) (at 53.34 109.22 90)
+      (effects (font (size 1.27 1.27)) hide)
+    )
     (pin "1")
     (pin "2")
@@
   )
   (symbol (lib_id "Device:C") (at 143.51 144.78 0) (unit 1)
-    (in_bom yes) (on_board yes) (fields_autoplaced)
-    (property "Reference" "C3" (id 0) (at 147.32 143.5099 0)
-      (effects (font (size 1.27 1.27)) (justify left))
-    )
-    (property "Value" "100nF" (id 1) (at 147.32 146.0499 0)
-      (effects (font (size 1.27 1.27)) (justify left) hide)
+    (in_bom yes) (on_board yes)
+    (property "Reference" "C3" (id 0) (at 139.7 142.24 0)
+      (effects (font (size 1.27 1.27)) (justify left))
+    )
+    (property "Value" "100nF" (id 1) (at 135.89 139.7 0)
+      (effects (font (size 1.27 1.27)) (justify left))
     )
     (property "Footprint" "Capacitor_SMD:C_0805_2012Metric_Pad1.18x1.45mm_HandSolder" (id 2) (at 144.4752 148.59 0)
@@
     )
     (property "Datasheet" "~" (id 3) (at 143.51 144.78 0)
+      (effects (font (size 1.27 1.27)) hide)
+    )
+    (property "Variant" "" (id 4) (at 143.51 144.78 0)
       (effects (font (size 1.27 1.27)) hide)
     )
@@
       (effects (font (size 1.27 1.27)) hide)
     )
+    (property "Variant" "B" (id 4) (at 143.51 179.07 90)
+      (effects (font (size 1.27 1.27)) hide)
+    )
     (pin "1")
     (pin "2")
@@
     )
     (property "Datasheet" " ~" (id 3) (at 133.35 57.15 0)
+      (effects (font (size 1.27 1.27)) hide)
+    )
+    (property "Variant" "A,B" (id 4) (at 133.35 57.15 0)
       (effects (font (size 1.27 1.27)) hide)
     )
@@
       (effects (font (size 1.27 1.27)) hide)
     )
+    (property "Variant" "B" (id 4) (at 52.07 119.38 0)
+      (effects (font (size 1.27 1.27)) hide)
+    )
     (pin "1")
     (pin "2")
@@
     )
     (path "/8422b3d4-486e-4fcf-a47a-02bf73d364a6"
-      (reference "L3") (unit 1) (value "?H") (footprint "Inductor_SMD:L_0805_2012Metric_Pad1.15x1.40mm_HandSolder")
+      (reference "L3") (unit 1) (value "1.2uH") (footprint "Inductor_SMD:L_0805_2012Metric_Pad1.15x1.40mm_HandSolder")
     )
     (path "/4f96ea1f-44c1-4973-933a-57d8b3b1bc93"

Commit message: ibom improved
Parts:
- C1, C11, C4, U2, U4: Variant (none) -> VarB
- C12, C2, C8, C9, J3, R13, R14, R15, R16, R4, R5: Variant B -> VarB
- C13, C5, J2, L1, U1: Variant A,B -> VarA,VarB
- R7, R8, XA1: Variant A -> VarA
Changed lines of the file:
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@@
+      (effects (font (size 1.27 1.27)) hide)
+    )
+    (property "Variant" "VarB" (id 4) (at 96.52 149.86 0)
       (effects (font (size 1.27 1.27)) hide)
     )
@@
       (effects (font (size 1.27 1.27)) hide)
     )
-    (property "Variant" "A,B" (id 4) (at 19.05 60.96 0)
+    (property "Variant" "VarA,VarB" (id 4) (at 19.05 60.96 0)
       (effects (font (size 1.27 1.27)) hide)
     )
@@
       (effects (font (size 1.27 1.27)) hide)
     )
-    (property "Variant" "B" (id 4) (at 60.96 105.41 0)
+    (property "Variant" "VarB" (id 4) (at 60.96 105.41 0)
       (effects (font (size 1.27 1.27)) hide)
     )
@@
       (effects (font (size 1.27 1.27)) hide)
     )
-    (property "Variant" "A,B" (id 4) (at 64.77 39.37 0)
+    (property "Variant" "VarA,VarB" (id 4) (at 64.77 39.37 0)
       (effects (font (size 1.27 1.27)) hide)
     )
@@
       (effects (font (size 1.27 1.27)) hide)
     )
-    (property "Variant" "A" (id 4) (at 163.83 25.4 90)
+    (property "Variant" "VarA" (id 4) (at 163.83 25.4 90)
       (effects (font (size 1.27 1.27)) hide)
     )
@@
       (effects (font (size 1.27 1.27)) hide)
     )
+    (property "Variant" "VarB" (id 4) (at 196.85 147.32 0)
+      (effects (font (size 1.27 1.27)) hide)
+    )
     (pin "1")
     (pin "2")
@@
       (effects (font (size 1.27 1.27)) hide)
     )
-    (property "Variant" "B" (id 4) (at 57.15 116.84 0)
+    (property "Variant" "VarB" (id 4) (at 57.15 116.84 0)
       (effects (font (size 1.27 1.27)) hide)
     )
@@
       (effects (font (size 1.27 1.27)) hide)
     )
-    (property "Variant" "B" (id 4) (at 57.15 181.61 0)
+    (property "Variant" "VarB" (id 4) (at 57.15 181.61 0)
       (effects (font (size 1.27 1.27)) hide)
     )
@@
       (effects (font (size 1.524 1.524)) hide)
     )
-    (property "Variant" "A" (id 4) (at 214.63 49.53 0)
+    (property "Variant" "VarA" (id 4) (at 214.63 49.53 0)
       (effects (font (size 1.27 1.27)) hide)
     )
@@
       (effects (font (size 1.27 1.27)) hide)
     )
-    (property "Variant" "B" (id 4) (at 168.91 137.16 0)
+    (property "Variant" "VarB" (id 4) (at 168.91 137.16 0)
       (effects (font (size 1.27 1.27)) hide)
     )
@@
       (effects (font (size 1.27 1.27)) hide)
     )
-    (property "Variant" "A" (id 4) (at 170.18 22.86 90)
+    (property "Variant" "VarA" (id 4) (at 170.18 22.86 90)
       (effects (font (size 1.27 1.27)) hide)
     )
@@
       (effects (font (size 1.27 1.27)) hide)
     )
-    (property "Variant" "A,B" (id 4) (at 111.76 53.34 0)
+    (property "Variant" "VarA,VarB" (id 4) (at 111.76 53.34 0)
       (effects (font (size 1.27 1.27)) hide)
     )
@@
       (effects (font (size 1.27 1.27)) hide)
     )
-    (property "Variant" "B" (id 4) (at 148.59 144.78 0)
+    (property "Variant" "VarB" (id 4) (at 148.59 144.78 0)
       (effects (font (size 1.27 1.27)) hide)
     )
@@
       (effects (font (size 1.27 1.27)) hide)
     )
-    (property "Variant" "B" (id 4) (at 138.43 149.86 90)
+    (property "Variant" "VarB" (id 4) (at 138.43 149.86 90)
       (effects (font (size 1.27 1.27)) hide)
     )
@@
       (effects (font (size 1.27 1.27)) hide)
     )
+    (property "Variant" "VarB" (id 4) (at 210.82 151.13 0)
+      (effects (font (size 1.27 1.27)) hide)
+    )
     (pin "1")
     (pin "2")
@@
       (effects (font (size 1.27 1.27)) hide)
     )
-    (property "Variant" "B" (id 4) (at 162.56 149.86 0)
+    (property "Variant" "VarB" (id 4) (at 162.56 149.86 0)
       (effects (font (size 1.27 1.27)) hide)
     )
@@
       (effects (font (size 1.27 1.27)) hide)
     )
-    (property "Variant" "B" (id 4) (at 138.43 152.4 90)
+    (property "Variant" "VarB" (id 4) (at 138.43 152.4 90)
       (effects (font (size 1.27 1.27)) hide)
     )
@@
     )
     (property "Datasheet" "~" (id 3) (at 205.74 151.13 0)
+      (effects (font (size 1.27 1.27)) hide)
+    )
+    (property "Variant" "VarB" (id 4) (at 205.74 151.13 0)
       (effects (font (size 1.27 1.27)) hide)
     )
@@
       (effects (font (size 1.27 1.27)) hide)
     )
-    (property "Variant" "A,B" (id 4) (at 30.48 60.96 0)
+    (property "Variant" "VarA,VarB" (id 4) (at 30.48 60.96 0)
       (effects (font (size 1.27 1.27)) hide)
     )
@@
       (effects (font (size 1.27 1.27)) hide)
     )
-    (property "Variant" "B" (id 4) (at 53.34 109.22 90)
+    (property "Variant" "VarB" (id 4) (at 53.34 109.22 90)
       (effects (font (size 1.27 1.27)) hide)
     )
@@
     )
     (property "Datasheet" "~" (id 3) (at 186.69 151.13 0)
+      (effects (font (size 1.27 1.27)) hide)
+    )
+    (property "Variant" "VarB" (id 4) (at 186.69 151.13 0)
       (effects (font (size 1.27 1.27)) hide)
     )
@@
       (effects (font (size 1.27 1.27)) hide)
     )
-    (property "Variant" "B" (id 4) (at 143.51 179.07 90)
+    (property "Variant" "VarB" (id 4) (at 143.51 179.07 90)
       (effects (font (size 1.27 1.27)) hide)
     )
@@
       (effects (font (size 1.27 1.27)) hide)
     )
-    (property "Variant" "A,B" (id 4) (at 133.35 57.15 0)
+    (property "Variant" "VarA,VarB" (id 4) (at 133.35 57.15 0)
       (effects (font (size 1.27 1.27)) hide)
     )
@@
       (effects (font (size 1.27 1.27)) hide)
     )
-    (property "Variant" "B" (id 4) (at 52.07 119.38 0)
-      (effects (font (size 1.27 1.27)) hide)
-    )
+    (property "Variant" "VarB" (id 4) (at 52.07 119.38 0)
+      (effects (font (size 1.27 1.27)) hide)
+    )

Commit message: ibom updated
Parts:
- C2: value 100nF -> 100pF
- C3: value 100nF -> 100pF; Variant (none) -> VarB
Changed lines of the file:
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@@
       (effects (font (size 1.27 1.27)) (justify left))
     )
-    (property "Value" "100nF" (id 1) (at 148.59 139.7 0)
+    (property "Value" "100pF" (id 1) (at 148.59 139.7 0)
       (effects (font (size 1.27 1.27)) (justify left))
     )
@@
       (effects (font (size 1.27 1.27)) (justify left))
     )
-    (property "Value" "100nF" (id 1) (at 135.89 139.7 0)
+    (property "Value" "100pF" (id 1) (at 135.89 139.7 0)
       (effects (font (size 1.27 1.27)) (justify left))
     )
@@
       (effects (font (size 1.27 1.27)) hide)
     )
-    (property "Variant" "" (id 4) (at 143.51 144.78 0)
+    (property "Variant" "VarB" (id 4) (at 143.51 144.78 0)
       (effects (font (size 1.27 1.27)) hide)
     )
@@
     )
     (path "/9ded86a2-fe8f-42cf-b17b-a865ec665344"
-      (reference "C2") (unit 1) (value "100nF") (footprint "Capacitor_SMD:C_0805_2012Metric_Pad1.18x1.45mm_HandSolder")
+      (reference "C2") (unit 1) (value "100pF") (footprint "Capacitor_SMD:C_0805_2012Metric_Pad1.18x1.45mm_HandSolder")
     )
     (path "/d4117451-fd31-4690-b77b-9a0d70931b45"
-      (reference "C3") (unit 1) (value "100nF") (footprint "Capacitor_SMD:C_0805_2012Metric_Pad1.18x1.45mm_HandSolder")
+      (reference "C3") (unit 1) (value "100pF") (footprint "Capacitor_SMD:C_0805_2012Metric_Pad1.18x1.45mm_HandSolder")
     )
     (path "/b8c17fd0-ceda-45fe-b025-f6c38eda4618"
