File: RTK1010Board.kicad_sch (KiCad schematic)
At the start: 75 parts, among them J1 SMA, J2 IPEX, J3 USB_OTG, J4 BNO055, U1 RTK-1010, U2 NCP1117-3.3_SOT223, U3 MCP1700-3302E_SOT23, U4 ESP32-S2-WROVER

Commit message: V1.0
Parts:
- added J5: Conn_GPS, footprints:CONN-TE-MICROMATCH-4X2-SMD, symbol Connector_Generic:Conn_01x08
- added TP_IO1, TP_IO17, TP_IO21, TP_IO26: TestPoint, TestPoint:TestPoint_Pad_D2.0mm, symbol Connector:TestPoint
- C10, C6, C7, L2, U3: Variant (none) -> OptD
Connections:
- net +3V3: now also J5.5 (Pin_5)
- net GND: now also J5.6 (Pin_6)
- net at U4.20 (ADC2_CH7/DAC_2/GPIO17): now also TP_IO17.1
- net at U4.24 (GPIO21): now also TP_IO21.1
- net at U4.25 (SPI_CS1/GPIO26): now also TP_IO26.1
- net GPS_RXD: now reaches U4.27 (GPIO33)
- net GPS_RXD: now also J5.1 (Pin_1)
- net GPS_SCL: now reaches U4.28 (GPIO34)
- net GPS_SCL: now also J5.2 (Pin_2)
- net GPS_TXD: now reaches U4.29 (GPIO35)
- net GPS_TXD: now also J5.3 (Pin_3)
- net GPS_SDA: now reaches U4.30 (GPIO36)
- net GPS_SDA: now also J5.4 (Pin_4)
- net GPS_7: now reaches U4.31 (GPIO37)
- net GPS_7: now also J5.7 (Pin_7)
- net GPS_8: now reaches U4.32 (GPIO38)
- net GPS_8: now also J5.8 (Pin_8)
- net at U4.39 (GPIO45): now also TP_IO1.1
Other:
- note added: "GPS Connector (Optional)"

Commit message: esp32_fw added
Parts:
- R15: value 100 -> 10k
Changed lines of the file:
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@@
     (in_bom yes) (on_board yes)
     (property "Reference" "R15" (id 0) (at 53.34 106.68 90))
-    (property "Value" "100" (id 1) (at 53.34 109.22 90))
+    (property "Value" "10k" (id 1) (at 53.34 109.22 90))
     (property "Footprint" "Resistor_SMD:R_0805_2012Metric_Pad1.20x1.40mm_HandSolder" (id 2) (at 53.34 107.442 90)
       (effects (font (size 1.27 1.27)) hide)
@@
     )
     (path "/c299d71a-84e4-40f7-9ee1-677d209cfe81"
-      (reference "R15") (unit 1) (value "100") (footprint "Resistor_SMD:R_0805_2012Metric_Pad1.20x1.40mm_HandSolder")
+      (reference "R15") (unit 1) (value "10k") (footprint "Resistor_SMD:R_0805_2012Metric_Pad1.20x1.40mm_HandSolder")
     )
     (path "/d4656162-6d2b-4fad-bd7b-1cd330016fb1"

Commit message: bom added
Parts:
- U4: OrderURL (none) -> https://www.reichelt.de/wifi-modul-802-11-bt-2-4-2-5ghz-150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
Changed lines of the file:
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@@
+      (effects (font (size 1.27 1.27)) hide)
+    )
+    (property "OrderURL" "https://www.reichelt.de/wifi-modul-802-11-bt-2-4-2-5ghz-150mb-s-esp32s2wroveri4-p311738.html?search=ESP32+S2+w" (id 5) (at 96.52 149.86 0)
       (effects (font (size 1.27 1.27)) hide)
     )
@@
       (effects (font (size 1.27 1.27)) hide)
     )
-    (property "Datasheet" "https://www.reichelt.de/usb-buchse-typ-micro-b-smd-gull-wing-mpe-712-1-s-bs0-p263308.html?&trstct=pol_1&nbc=1" (id 3) (at 158.75 151.13 0)
-      (effects (font (size 1.27 1.27)) hide)
-    )
+    (property "Datasheet" "https://www.mouser.de/ProductDetail/Amphenol-FCI/10118194-0001LF?qs=Ywefl8B65e4FIdY8OWfRQA%3D%3D" (id 3) (at 158.75 151.13 0)
+      (effects (font (size 1.27 1.27)) hide)
+    )
